File: eeZee_microSD/eeZee microSD.sch (EAGLE design)
At the start: 19 parts, among them U1 MCP1824S, U2 74HC4050

Commit message: Fixes to PropVGA, microSD,
Parts:
- removed LED1, LED2: (no value), mes_opto:LEDCHIPLED_0805
- removed R1, R2: 1K, rcl:R-US_R0603
Connections:
- removed net N$1: LED2.A, R2.1
- removed net N$2: LED1.A, R1.1
- net GND: no longer LED1.C, LED2.C
- net SCK_HV: no longer R1.2
- net VBOARD: no longer R2.2
Changed lines of the file:
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@@
 <grid distance="0.1" unitdist="inch" unit="inch" style="lines" multiple="1" display="no" altdistance="0.01" altunitdist="inch" altunit="inch"/>
 <layers>
-<layer number="1" name="Top" color="4" fill="1" visible="yes" active="no"/>
-<layer number="16" name="Bottom" color="1" fill="1" visible="yes" active="no"/>
-<layer number="17" name="Pads" color="2" fill="1" visible="yes" active="no"/>
-<layer number="18" name="Vias" color="2" fill="1" visible="yes" active="no"/>
-<layer number="19" name="Unrouted" color="6" fill="1" visible="yes" active="no"/>
-<layer number="20" name="Dimension" color="15" fill="1" visible="yes" active="no"/>
-<layer number="21" name="tPlace" color="7" fill="1" visible="yes" active="no"/>
-<layer number="22" name="bPlace" color="7" fill="1" visible="yes" active="no"/>
-<layer number="23" name="tOrigins" color="15" fill="1" visible="yes" active="no"/>
-<layer number="24" name="bOrigins" color="15" fill="1" visible="yes" active="no"/>
-<layer number="25" name="tNames" color="7" fill="1" visible="yes" active="no"/>
-<layer number="26" name="bNames" color="7" fill="1" visible="yes" active="no"/>
-<layer number="27" name="tValues" color="7" fill="1" visible="yes" active="no"/>
-<layer number="28" name="bValues" color="7" fill="1" visible="yes" active="no"/>
+<layer number="1" name="Top" color="4" fill="1" visible="no" active="no"/>
+<layer number="16" name="Bottom" color="1" fill="1" visible="no" active="no"/>
+<layer number="17" name="Pads" color="2" fill="1" visible="no" active="no"/>
+<layer number="18" name="Vias" color="2" fill="1" visible="no" active="no"/>
+<layer number="19" name="Unrouted" color="6" fill="1" visible="no" active="no"/>
+<layer number="20" name="Dimension" color="15" fill="1" visible="no" active="no"/>
+<layer number="21" name="tPlace" color="7" fill="1" visible="no" active="no"/>
+<layer number="22" name="bPlace" color="7" fill="1" visible="no" active="no"/>
+<layer number="23" name="tOrigins" color="15" fill="1" visible="no" active="no"/>
+<layer number="24" name="bOrigins" color="15" fill="1" visible="no" active="no"/>
+<layer number="25" name="tNames" color="7" fill="1" visible="no" active="no"/>
+<layer number="26" name="bNames" color="7" fill="1" visible="no" active="no"/>
+<layer number="27" name="tValues" color="7" fill="1" visible="no" active="no"/>
+<layer number="28" name="bValues" color="7" fill="1" visible="no" active="no"/>
 <layer number="29" name="tStop" color="7" fill="3" visible="no" active="no"/>
 <layer number="30" name="bStop" color="7" fill="6" visible="no" active="no"/>
@@
 <layer number="35" name="tGlue" color="7" fill="4" visible="no" active="no"/>
 <layer number="36" name="bGlue" color="7" fill="5" visible="no" active="no"/>
-<layer number="37" name="tTest" color="7" fill="1" visible="yes" active="no"/>
-<layer number="38" name="bTest" color="7" fill="1" visible="yes" active="no"/>
+<layer number="37" name="tTest" color="7" fill="1" visible="no" active="no"/>
+<layer number="38" name="bTest" color="7" fill="1" visible="no" active="no"/>
 <layer number="39" name="tKeepout" color="4" fill="11" visible="no" active="no"/>
 <layer number="40" name="bKeepout" color="1" fill="11" visible="no" active="no"/>
@@
 <layer number="44" name="Drills" color="7" fill="1" visible="no" active="no"/>
 <layer number="45" name="Holes" color="7" fill="1" visible="no" active="no"/>
-<layer number="46" name="Milling" color="3" fill="1" visible="yes" active="no"/>
-<layer number="47" name="Measures" color="7" fill="1" visible="yes" active="no"/>
-<layer number="48" name="Document" color="7" fill="1" visible="yes" active="no"/>
-<layer number="49" name="Reference" color="7" fill="1" visible="yes" active="no"/>
-<layer number="50" name="dxf" color="7" fill="1" visible="yes" active="no"/>
-<layer number="51" name="tDocu" color="11" fill="1" visible="yes" active="no"/>
-<layer number="52" name="bDocu" color="7" fill="1" visible="yes" active="no"/>
-<layer number="53" name="tGND_GNDA" color="7" fill="9" visible="yes" active="no"/>
-<layer number="54" name="bGND_GNDA" color="1" fill="9" visible="yes" active="no"/>
-<layer number="56" name="wert" color="7" fill="1" visible="yes" active="no"/>
+<layer number="46" name="Milling" color="3" fill="1" visible="no" active="no"/>
+<layer number="47" name="Measures" color="7" fill="1" visible="no" active="no"/>
+<layer number="48" name="Document" color="7" fill="1" visible="no" active="no"/>
+<layer number="49" name="Reference" color="7" fill="1" visible="no" active="no"/>
+<layer number="50" name="dxf" color="7" fill="1" visible="no" active="no"/>
+<layer number="51" name="tDocu" color="11" fill="1" visible="no" active="no"/>
+<layer number="52" name="bDocu" color="7" fill="1" visible="no" active="no"/>
+<layer number="53" name="tGND_GNDA" color="7" fill="9" visible="no" active="no"/>
+<layer number="54" name="bGND_GNDA" color="1" fill="9" visible="no" active="no"/>
+<layer number="56" name="wert" color="7" fill="1" visible="no" active="no"/>
 <layer number="91" name="Nets" color="2" fill="1" visible="yes" active="yes"/>
 <layer number="92" name="Busses" color="1" fill="1" visible="yes" active="yes"/>
@@
 <attribute name="PARTNO" value="LMK107B7105KA-T"/>
 </part>
-<part name="LED1" library="mes_opto" deviceset="LED" device="CHIPLED_0805"/>
-<part name="R1" library="rcl" deviceset="R-US_" device="R0603" value="1K">
-<attribute name="PARTNO" value="ERJ-3GEYJ103V"/>
-</part>
 <part name="GND5" library="mes" deviceset="GND" device=""/>
 <part name="JP3" library="mes_electromech" deviceset="PINHEAD-2" device="BIG" value="PWR"/>
@@
 <part name="JP5" library="mes_electromech" deviceset="PINHEAD-2" device="BIG" value="PWR"/>
 <part name="JP4" library="mes_electromech" deviceset="PINHEAD-2" device="BIG" value="PWR"/>
-<part name="R2" library="rcl" deviceset="R-US_" device="R0603" value="1K">
-<attribute name="PARTNO" value="ERJ-3GEYJ103V"/>
-</part>
-<part name="LED2" library="mes_opto" deviceset="LED" device="CHIPLED_0805"/>
 </parts>
 <sheets>
@@
 <attribute name="PARTNO" value="JMK212BJ226MG-T" x="170.18" y="101.6" size="1.778" layer="96" display="off"/>
 </instance>
-<instance part="LED1" gate="G$1" x="127" y="50.8"/>
-<instance part="R1" gate="G$1" x="127" y="60.96" rot="R90">
-<attribute name="PARTNO" value="ERJ-3GEYJ102V" x="127" y="60.96" size="1.778" layer="96" rot="R90" display="off"/>
-</instance>
-<instance part="GND5" gate="1" x="127" y="38.1"/>
+<instance part="GND5" gate="1" x="106.68" y="38.1"/>
 <instance part="JP3" gate="JP1" x="190.5" y="99.06"/>
 <instance part="JP2" gate="JP1" x="190.5" y="111.76"/>
 <instance part="JP5" gate="JP1" x="190.5" y="73.66"/>
 <instance part="JP4" gate="JP1" x="190.5" y="86.36"/>
-<instance part="R2" gate="G$1" x="160.02" y="106.68" rot="R90">
-<attribute name="PARTNO" value="ERJ-3GEYJ102V" x="160.02" y="106.68" size="1.778" layer="96" rot="R90" display="off"/>
-</instance>
-<instance part="LED2" gate="G$1" x="160.02" y="96.52"/>
 </instances>
 <busses>
@@
 <net name="SCK_HV" class="0">
 <segment>
-<wire x1="154.94" y1="71.12" x2="127" y2="71.12" width="0.1524" layer="91"/>
 <pinref part="JP6" gate="A" pin="1"/>
 <label x="137.16" y="71.12" size="1.778" layer="95"/>
 <pinref part="U2" gate="G$1" pin="4A"/>
-<wire x1="99.06" y1="71.12" x2="127" y2="71.12" width="0.1524" layer="91"/>
-<pinref part="R1" gate="G$1" pin="2"/>
-<wire x1="127" y1="66.04" x2="127" y2="71.12" width="0.1524" layer="91"/>
-<junction x="127" y="71.12"/>
+<wire x1="99.06" y1="71.12" x2="154.94" y2="71.12" width="0.1524" layer="91"/>
 <label x="119.38" y="71.12" size="1.778" layer="95" rot="MR0"/>
 </segment>
@@
 <junction x="55.88" y="58.42"/>
 <pinref part="GND5" gate="1" pin="GND"/>
-<pinref part="LED1" gate="G$1" pin="C"/>
-<wire x1="127" y1="40.64" x2="127" y2="43.18" width="0.1524" layer="91"/>
-<wire x1="127" y1="43.18" x2="127" y2="45.72" width="0.1524" layer="91"/>
+<wire x1="106.68" y1="40.64" x2="106.68" y2="43.18" width="0.1524" layer="91"/>
 <wire x1="55.88" y1="43.18" x2="76.2" y2="43.18" width="0.1524" layer="91"/>
 <pinref part="U2" gate="G$1" pin="GND"/>
 <wire x1="76.2" y1="43.18" x2="101.6" y2="43.18" width="0.1524" layer="91"/>
 <wire x1="101.6" y1="43.18" x2="106.68" y2="43.18" width="0.1524" layer="91"/>
-<wire x1="106.68" y1="43.18" x2="127" y2="43.18" width="0.1524" layer="91"/>
 <wire x1="78.74" y1="81.28" x2="76.2" y2="81.28" width="0.1524" layer="91"/>
 <wire x1="76.2" y1="81.28" x2="76.2" y2="43.18" width="0.1524" layer="91"/>
@@
 <wire x1="106.68" y1="55.88" x2="106.68" y2="43.18" width="0.1524" layer="91"/>
 <junction x="106.68" y="43.18"/>
-<junction x="127" y="43.18"/>
+<junction x="106.68" y="43.18"/>
 </segment>
 <segment>
@@
 <junction x="177.8" y="124.46"/>
 <wire x1="177.8" y1="86.36" x2="170.18" y2="86.36" width="0.1524" layer="91"/>
-<wire x1="170.18" y1="86.36" x2="160.02" y2="86.36" width="0.1524" layer="91"/>
 <wire x1="170.18" y1="96.52" x2="170.18" y2="86.36" width="0.1524" layer="91"/>
-<junction x="170.18" y="86.36"/>
-<pinref part="LED2" gate="G$1" pin="C"/>
-<wire x1="160.02" y1="86.36" x2="160.02" y2="91.44" width="0.1524" layer="91"/>
 </segment>
 </net>
@@
 <wire x1="170.18" y1="114.3" x2="160.02" y2="114.3" width="0.1524" layer="91"/>
 <junction x="170.18" y="114.3"/>
-<label x="160.02" y="114.3" size="1.778" layer="95"/>
-<pinref part="R2" gate="G$1" pin="2"/>
-<wire x1="160.02" y1="111.76" x2="160.02" y2="114.3" width="0.1524" layer="91"/>
+<label x="162.56" y="114.3" size="1.778" layer="95"/>
 </segment>
 </net>
@@
 </segment>
 </net>
-<net name="N$1" class="0">
-<segment>
-<pinref part="LED2" gate="G$1" pin="A"/>
-<pinref part="R2" gate="G$1" pin="1"/>
-<wire x1="160.02" y1="101.6" x2="160.02" y2="99.06" width="0.1524" layer="91"/>
-</segment>
-</net>
-<net name="N$2" class="0">
-<segment>
-<pinref part="LED1" gate="G$1" pin="A"/>
-<pinref part="R1" gate="G$1" pin="1"/>
-<wire x1="127" y1="53.34" x2="127" y2="55.88" width="0.1524" layer="91"/>
-</segment>
-</net>
